File: MacOS Keyboard/correct pcd setup/correct pcd setup.kicad_pcb (KiCad board)
At the start: 4 copper layers, 437 parts, among them J1 USB_C, SW1 SW_Push, U1 74AHCT125, U2 STM32F072CBTx, U3 XC6206, U4 USBLC6-2SC6

Commit message: things
Parts:
- added C10: 100nF, ScottoKeebs_Components:Capacitor_0402, F.Cu at (535.4, 340.6)
- added C11: 100nF, ScottoKeebs_Components:Capacitor_0402, F.Cu at (544.2, 331.7)
- added C12: 4.7uF, ScottoKeebs_Components:Capacitor_0402, F.Cu at (544.2, 330.7)
- added C13: 100nF, ScottoKeebs_Components:Capacitor_0402, F.Cu at (532.0, 337.2)
- added C14: 10nF, ScottoKeebs_Components:Capacitor_0402, F.Cu at (539.1, 340.6)
- added C15: 1uF, ScottoKeebs_Components:Capacitor_0402, F.Cu at (540.1, 340.6)
- added C16: 100nF, ScottoKeebs_Components:Capacitor_0402, F.Cu at (534.4, 329.7)
- added C17: 4.7uF, ScottoKeebs_Components:Capacitor_0402, F.Cu at (533.4, 329.7)
- added C7: 100nF, ScottoKeebs_Components:Capacitor_0402, F.Cu at (538.1, 340.6)
- added C8: 1uF, ScottoKeebs_Components:Capacitor_0402, F.Cu at (533.2, 313.3)
- added C9: 1uF, ScottoKeebs_Components:Capacitor_0402, F.Cu at (534.1, 318.2)
- added F1: 500mA, ScottoKeebs_Components:Fuse_0603, F.Cu at (532.9, 312.1)
- added J1: USB_C, ScottoKeebs_Components:USB_C_HRO_TYPE-C-31-M-12, F.Cu at (536.6, 296.6)
- added R1: 10k, ScottoKeebs_Components:Resistor_0402, F.Cu at (547.9, 314.5)
- added R2: 5.1k, ScottoKeebs_Components:Resistor_0402, F.Cu at (538.4, 303.3)
- added R3: 5.1k, ScottoKeebs_Components:Resistor_0402, F.Cu at (534.9, 303.1)
- added SW1: SW_Push, ScottoKeebs_Components:Button_TL3342, F.Cu at (543.1, 315.8)
- added U1: STM32F072CBT6, ScottoKeebs_Components:Package_LQFP-48_7x7mm_P0.5, F.Cu at (538.1, 334.5)
- added U3: XC6206, ScottoKeebs_Components:Voltage_SOT-23, F.Cu at (533.7, 315.7)
- added U4: USBLC6-2SC6, ScottoKeebs_Components:ESD_SOT-23-6, F.Cu at (537.1, 310.7)
- U2: moved to F.Cu
- moved J1 674.7 mm to (502.7, 274.7), turned to 180 degrees
- moved R1 657.0 mm to (521.4, 237.8)
- moved R2 657.0 mm to (521.4, 239.8)
- moved R3 657.0 mm to (521.4, 241.8)
- moved U3 657.0 mm to (522.4, 245.0)
- moved F1 657.0 mm to (521.9, 248.5)
- moved RV1 657.0 mm to (526.6, 232.6)
- moved SW1 657.0 mm to (513.4, 245.7)
- moved U4 657.0 mm to (525.4, 239.1)
- moved U2 339.7 mm to (502.7, 331.8), turned to 90 degrees
- moved C100 316.4 mm to (152.3, 58.3)
- moved C101 316.4 mm to (152.3, 60.3)
- moved C102 316.4 mm to (152.3, 62.2)
- moved C103 316.4 mm to (152.3, 64.2)
- moved C104 316.4 mm to (152.3, 66.2)
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Connections:
- D51 pad 1: A7 -> unconnected-(D51-K-Pad1)
Routing:
- net +3.3V: track 27.0 -> 98.4 mm, vias 0 -> 7
- net /BOOT0: track 0.00 -> 34.8 mm, vias 0 -> 2
- net VBUS: track 0.00 -> 32.8 mm, vias 0 -> 3
- net GND: track 0.00 -> 24.6 mm, vias 0 -> 20
- net /MCU_D-: track 0.00 -> 18.6 mm
- net /MCU_D+: track 0.00 -> 18.6 mm
- net /USB_D+: track 0.00 -> 16.4 mm
- net /USB_D-: track 0.00 -> 12.2 mm
- net /D-: track 0.00 -> 10.5 mm
- net Net-(J1-CC1): track 0.00 -> 5.20 mm
- net Net-(J1-CC2): track 0.00 -> 3.92 mm
- net /D+: track 0.00 -> 2.83 mm
- net +5V: track 0.00 -> 2.76 mm
- net /NRST: track 0.00 -> 1.54 mm
- added copper zone on F.Cu, net /USB_D+
- added copper zone on B.Cu, net VBUS
Other:
- board outline added: 513.3 x 324.2 mm
- board text added: "JLCJLCJLCJLC"
