File: MacOS Keyboard/STM32F072CBT6/_autosave-ScottoModules.kicad_pcb (KiCad board)
At the start: 4 copper layers, 436 parts, among them J1 USB_C, SW1 SW_Push, SW2 RotaryEncoder, U1 STM32F072CBTx, U2 74AHCT125, U3 XC6206, U4 USBLC6-2SC6

Commit message: changes
Parts:
- removed the R2 at (-54.0, 39.4)
- removed the R2 at (-48.1, 3.24)
- removed the R3 at (-44.5, 3.12)
- added R2: 5.1k, ScottoKeebs_Components:Resistor_0402, B.Cu at (21.1, 0.84)
- DisplayLED1, DisplayLED2, DisplayLED3, LEDBULKCAP1, R3, R4: moved to B.Cu
- DisplayLEDCAP2: renamed from DisplayLEDCAP1; moved to B.Cu
- DisplayLEDCAP3: renamed from DisplayLEDCAP2; moved to B.Cu
- moved DisplayLED3 668.5 mm to (412.1, 38.1), turned to 180 degrees
- moved DisplayLED2 632.5 mm to (390.6, 38.1), turned to 180 degrees
- moved DisplayLEDCAP3 618.2 mm to (407.5, 38.1), turned to -90 degrees
- moved DisplayLED1 607.7 mm to (369.1, 38.1), turned to 180 degrees
- moved DisplayLEDCAP2 598.1 mm to (386.0, 38.1), turned to -90 degrees
- moved SW2 528.5 mm to (438.3, 35.6)
- moved DisplayLEDCAP1 445.4 mm to (364.4, 38.1), turned to -90 degrees
- moved R3 396.7 mm to (24.7, 1.16), turned to -90 degrees
- moved R4 338.6 mm to (33.3, 44.1)
- moved LEDBULKCAP1 334.2 mm to (32.6, 42.5), turned to -90 degrees
- moved C10 69.3 mm to (24.2, 38.3)
- moved C11 69.3 mm to (15.4, 29.4)
- moved C12 69.3 mm to (15.4, 28.4)
- moved C13 69.3 mm to (27.6, 34.9)
- moved C14 69.3 mm to (20.5, 38.3)
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- renumbered DisplayLEDCAP102 to DisplayLEDCAP1
Routing:
- net GND: track 47810.3 -> 10.3 mm
- net A6: track 0.00 -> 428.1 mm
- net A7: track 0.00 -> 426.7 mm
- net A9: track 0.00 -> 415.6 mm
- net A10: track 0.00 -> 399.4 mm
- net A8: track 0.00 -> 397.6 mm
- net A5: track 0.00 -> 277.8 mm
- net A15: track 33.0 -> 0.00 mm
- net +5V: track 30.5 -> 6.27 mm
- net B10: track 138.0 -> 142.5 mm
- net B12: track 131.7 -> 135.8 mm
- net Net-(D96-A): track 6.97 -> 3.22 mm
- net Net-(D95-A): track 6.97 -> 3.22 mm
- net Net-(D94-A): track 6.97 -> 3.22 mm
- net Net-(D101-A): track 6.97 -> 3.22 mm
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