File: MacOS Keyboard/STM32F072CBT6/DiodePlacement.kicad_pcb (KiCad board)
At the start: 2 copper layers, 2 parts

Commit message: :P
Routing:
- net B0: track 0.00 -> 113.7 mm
Changed lines of the file:
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@@
 		(net 1)
+	)
+	(segment
+		(start -7.085 26.035)
+		(end -7.085 40.3225)
+		(width 0.2)
+		(layer "B.Cu")
+		(net 2)
+	)
+	(segment
+		(start -7.085 40.3225)
+		(end -2.3225 45.085)
+		(width 0.2)
+		(layer "B.Cu")
+		(net 2)
+	)
+	(segment
+		(start 0.05875 78.4225)
+		(end 4.82125 83.185)
+		(width 0.2)
+		(layer "B.Cu")
+		(net 2)
+	)
+	(segment
+		(start -2.3225 61.75375)
+		(end 0.05875 64.135)
+		(width 0.2)
+		(layer "B.Cu")
+		(net 2)
+	)
+	(segment
+		(start 4.82125 83.185)
+		(end -4.70375 92.71)
+		(width 0.2)
+		(layer "B.Cu")
+		(net 2)
+	)
+	(segment
+		(start -4.70375 92.71)
+		(end -4.70375 102.235)
+		(width 0.2)
+		(layer "B.Cu")
+		(net 2)
+	)
+	(segment
+		(start -7.085 -2.54)
+		(end -7.085 26.035)
+		(width 0.2)
+		(layer "B.Cu")
+		(net 2)
+	)
+	(segment
+		(start -2.3225 45.085)
+		(end -2.3225 61.75375)
+		(width 0.2)
+		(layer "B.Cu")
+		(net 2)
+	)
+	(segment
+		(start 0.05875 64.135)
+		(end 0.05875 78.4225)
+		(width 0.2)
+		(layer "B.Cu")
+		(net 2)
 	)
 	(embedded_fonts no)
