File: MacOS Keyboard/STM32F072CBT6/LED.kicad_sch (KiCad schematic)
At the start: 210 parts

Commit message: :P
Parts:
- added LEDBULKCAP2, LEDBULKCAP3, LEDBULKCAP4, LEDBULKCAP5, LEDBULKCAP6: 100uF, ScottoKeebs_Components:Capacitor_0402, symbol Device:C_Small
- added R5: 500R, ScottoKeebs_Components:Resistor_0402, symbol Device:R_Small
- DisplayLED1, DisplayLED2, DisplayLED3, LED1, LED10, LED100, LED101, LED11, LED12, LED13, LED14, LED15, LED16, LED17, LED18, LED19, LED2, LED20, LED21, LED22, LED23, LED24, LED25, LED26, LED27, LED28, LED29, LED3, LED30, LED31, LED32, LED33, LED34, LED35, LED36, LED37, LED38, LED39, LED4, LED40, LED41, LED42, LED43, LED44, LED45, LED46, LED47, LED48, LED49, LED5, LED50, LED51, LED52, LED53, LED54, LED55, LED56, LED57, LED58, LED59, LED6, LED60, LED61, LED62, LED63, LED64, LED65, LED66, LED67, LED68, LED69, LED7, LED70, LED71, LED72, LED73, LED74, LED75, LED76, LED77, LED78, LED79, LED8, LED80, LED81, LED82, LED83, LED84, LED85, LED86, LED87, LED88, LED89, LED9, LED90, LED91, LED92, LED93, LED94, LED95, LED96, LED97, LED98, LED99: footprint LED_SMD:LED_SK6812MINI_PLCC4_3.5x3.5mm_P1.75mm -> ScottoKeebs_Components:LED_SK6812MINI; symbol LED:SK6812MINI -> ScottoKeebs:LED_SK6812MINI; LCSC (none) -> C5149201
- R4: value 330R -> 500R
- renumbered DisplayLEDCAP102 to DisplayLEDCAP1, DisplayLEDCAP1 to DisplayLEDCAP2, DisplayLEDCAP2 to DisplayLEDCAP3
Connections:
- net 5V: now also DisplayLED1.1 (VDD), DisplayLED2.1 (VDD), DisplayLED3.1 (VDD), LED1.1 (VDD), LED10.1 (VDD), LED100.1 (VDD), LED101.1 (VDD), LED11.1 (VDD), LED12.1 (VDD), LED13.1 (VDD), LED14.1 (VDD), LED15.1 (VDD), LED16.1 (VDD), LED17.1 (VDD), LED18.1 (VDD), LED19.1 (VDD), LED2.1 (VDD), LED20.1 (VDD), LED21.1 (VDD), LED22.1 (VDD), LED23.1 (VDD), LED24.1 (VDD), LED25.1 (VDD), LED26.1 (VDD), LED27.1 (VDD), LED28.1 (VDD), LED29.1 (VDD), LED3.1 (VDD), LED30.1 (VDD), LED31.1 (VDD), LED32.1 (VDD), LED33.1 (VDD), LED34.1 (VDD), LED35.1 (VDD), LED36.1 (VDD), LED37.1 (VDD), LED38.1 (VDD), LED39.1 (VDD), LED4.1 (VDD), LED40.1 (VDD), LED41.1 (VDD), LED42.1 (VDD), LED43.1 (VDD), LED44.1 (VDD), LED45.1 (VDD), LED46.1 (VDD), LED47.1 (VDD), LED48.1 (VDD), LED49.1 (VDD), LED5.1 (VDD), LED50.1 (VDD), LED51.1 (VDD), LED52.1 (VDD), LED53.1 (VDD), LED54.1 (VDD), LED55.1 (VDD), LED56.1 (VDD), LED57.1 (VDD), LED58.1 (VDD), LED59.1 (VDD), LED6.1 (VDD), LED60.1 (VDD), LED61.1 (VDD), LED62.1 (VDD), LED63.1 (VDD), LED64.1 (VDD), LED65.1 (VDD), LED66.1 (VDD), LED67.1 (VDD), LED68.1 (VDD), LED69.1 (VDD), LED7.1 (VDD), LED70.1 (VDD), LED71.1 (VDD), LED72.1 (VDD), LED73.1 (VDD), LED74.1 (VDD), LED75.1 (VDD), LED76.1 (VDD), LED77.1 (VDD), LED78.1 (VDD), LED79.1 (VDD), LED8.1 (VDD), LED80.1 (VDD), LED81.1 (VDD), LED82.1 (VDD), LED83.1 (VDD), LED84.1 (VDD), LED85.1 (VDD), LED86.1 (VDD), LED87.1 (VDD), LED88.1 (VDD), LED89.1 (VDD), LED9.1 (VDD), LED90.1 (VDD), LED91.1 (VDD), LED92.1 (VDD), LED93.1 (VDD), LED94.1 (VDD), LED95.1 (VDD), LED96.1 (VDD), LED97.1 (VDD), LED98.1 (VDD), LED99.1 (VDD), LEDBULKCAP2.1, LEDBULKCAP3.1, LEDBULKCAP4.1, LEDBULKCAP5.1, LEDBULKCAP6.1; no longer DisplayLED1.4 (VDD), DisplayLED2.4 (VDD), DisplayLED3.4 (VDD), LED1.4 (VDD), LED10.4 (VDD), LED100.4 (VDD), LED101.4 (VDD), LED11.4 (VDD), LED12.4 (VDD), LED13.4 (VDD), LED14.4 (VDD), LED15.4 (VDD), LED16.4 (VDD), LED17.4 (VDD), LED18.4 (VDD), LED19.4 (VDD), LED2.4 (VDD), LED20.4 (VDD), LED21.4 (VDD), LED22.4 (VDD), LED23.4 (VDD), LED24.4 (VDD), LED25.4 (VDD), LED26.4 (VDD), LED27.4 (VDD), LED28.4 (VDD), LED29.4 (VDD), LED3.4 (VDD), LED30.4 (VDD), LED31.4 (VDD), LED32.4 (VDD), LED33.4 (VDD), LED34.4 (VDD), LED35.4 (VDD), LED36.4 (VDD), LED37.4 (VDD), LED38.4 (VDD), LED39.4 (VDD), LED4.4 (VDD), LED40.4 (VDD), LED41.4 (VDD), LED42.4 (VDD), LED43.4 (VDD), LED44.4 (VDD), LED45.4 (VDD), LED46.4 (VDD), LED47.4 (VDD), LED48.4 (VDD), LED49.4 (VDD), LED5.4 (VDD), LED50.4 (VDD), LED51.4 (VDD), LED52.4 (VDD), LED53.4 (VDD), LED54.4 (VDD), LED55.4 (VDD), LED56.4 (VDD), LED57.4 (VDD), LED58.4 (VDD), LED59.4 (VDD), LED6.4 (VDD), LED60.4 (VDD), LED61.4 (VDD), LED62.4 (VDD), LED63.4 (VDD), LED64.4 (VDD), LED65.4 (VDD), LED66.4 (VDD), LED67.4 (VDD), LED68.4 (VDD), LED69.4 (VDD), LED7.4 (VDD), LED70.4 (VDD), LED71.4 (VDD), LED72.4 (VDD), LED73.4 (VDD), LED74.4 (VDD), LED75.4 (VDD), LED76.4 (VDD), LED77.4 (VDD), LED78.4 (VDD), LED79.4 (VDD), LED8.4 (VDD), LED80.4 (VDD), LED81.4 (VDD), LED82.4 (VDD), LED83.4 (VDD), LED84.4 (VDD), LED85.4 (VDD), LED86.4 (VDD), LED87.4 (VDD), LED88.4 (VDD), LED89.4 (VDD), LED9.4 (VDD), LED90.4 (VDD), LED91.4 (VDD), LED92.4 (VDD), LED93.4 (VDD), LED94.4 (VDD), LED95.4 (VDD), LED96.4 (VDD), LED97.4 (VDD), LED98.4 (VDD), LED99.4 (VDD)
- net D1: now also DisplayLED3.2 (DOUT), LED14.4 (DIN); no longer DisplayLED3.1 (DOUT), LED14.3 (DIN)
- net D2: now also LED34.2 (DOUT), LED35.4 (DIN); no longer LED34.1 (DOUT), LED35.3 (DIN)
- net D3: now also LED55.2 (DOUT), LED56.4 (DIN); no longer LED55.1 (DOUT), LED56.3 (DIN)
- net D4: now also LED71.2 (DOUT), LED72.4 (DIN); no longer LED71.1 (DOUT), LED72.3 (DIN)
- net D5: now also LED88.2 (DOUT), LED89.4 (DIN); no longer LED88.1 (DOUT), LED89.3 (DIN)
- net GND: now also DisplayLED1.3 (VSS), DisplayLED2.3 (VSS), DisplayLED3.3 (VSS), LED1.3 (VSS), LED10.3 (VSS), LED100.3 (VSS), LED101.3 (VSS), LED11.3 (VSS), LED12.3 (VSS), LED13.3 (VSS), LED14.3 (VSS), LED15.3 (VSS), LED16.3 (VSS), LED17.3 (VSS), LED18.3 (VSS), LED19.3 (VSS), LED2.3 (VSS), LED20.3 (VSS), LED21.3 (VSS), LED22.3 (VSS), LED23.3 (VSS), LED24.3 (VSS), LED25.3 (VSS), LED26.3 (VSS), LED27.3 (VSS), LED28.3 (VSS), LED29.3 (VSS), LED3.3 (VSS), LED30.3 (VSS), LED31.3 (VSS), LED32.3 (VSS), LED33.3 (VSS), LED34.3 (VSS), LED35.3 (VSS), LED36.3 (VSS), LED37.3 (VSS), LED38.3 (VSS), LED39.3 (VSS), LED4.3 (VSS), LED40.3 (VSS), LED41.3 (VSS), LED42.3 (VSS), LED43.3 (VSS), LED44.3 (VSS), LED45.3 (VSS), LED46.3 (VSS), LED47.3 (VSS), LED48.3 (VSS), LED49.3 (VSS), LED5.3 (VSS), LED50.3 (VSS), LED51.3 (VSS), LED52.3 (VSS), LED53.3 (VSS), LED54.3 (VSS), LED55.3 (VSS), LED56.3 (VSS), LED57.3 (VSS), LED58.3 (VSS), LED59.3 (VSS), LED6.3 (VSS), LED60.3 (VSS), LED61.3 (VSS), LED62.3 (VSS), LED63.3 (VSS), LED64.3 (VSS), LED65.3 (VSS), LED66.3 (VSS), LED67.3 (VSS), LED68.3 (VSS), LED69.3 (VSS), LED7.3 (VSS), LED70.3 (VSS), LED71.3 (VSS), LED72.3 (VSS), LED73.3 (VSS), LED74.3 (VSS), LED75.3 (VSS), LED76.3 (VSS), LED77.3 (VSS), LED78.3 (VSS), LED79.3 (VSS), LED8.3 (VSS), LED80.3 (VSS), LED81.3 (VSS), LED82.3 (VSS), LED83.3 (VSS), LED84.3 (VSS), LED85.3 (VSS), LED86.3 (VSS), LED87.3 (VSS), LED88.3 (VSS), LED89.3 (VSS), LED9.3 (VSS), LED90.3 (VSS), LED91.3 (VSS), LED92.3 (VSS), LED93.3 (VSS), LED94.3 (VSS), LED95.3 (VSS), LED96.3 (VSS), LED97.3 (VSS), LED98.3 (VSS), LED99.3 (VSS), LEDBULKCAP2.2, LEDBULKCAP3.2, LEDBULKCAP4.2, LEDBULKCAP5.2, LEDBULKCAP6.2; no longer DisplayLED1.2 (VSS), DisplayLED2.2 (VSS), DisplayLED3.2 (VSS), LED1.2 (VSS), LED10.2 (VSS), LED100.2 (VSS), LED101.2 (VSS), LED11.2 (VSS), LED12.2 (VSS), LED13.2 (VSS), LED14.2 (VSS), LED15.2 (VSS), LED16.2 (VSS), LED17.2 (VSS), LED18.2 (VSS), LED19.2 (VSS), LED2.2 (VSS), LED20.2 (VSS), LED21.2 (VSS), LED22.2 (VSS), LED23.2 (VSS), LED24.2 (VSS), LED25.2 (VSS), LED26.2 (VSS), LED27.2 (VSS), LED28.2 (VSS), LED29.2 (VSS), LED3.2 (VSS), LED30.2 (VSS), LED31.2 (VSS), LED32.2 (VSS), LED33.2 (VSS), LED34.2 (VSS), LED35.2 (VSS), LED36.2 (VSS), LED37.2 (VSS), LED38.2 (VSS), LED39.2 (VSS), LED4.2 (VSS), LED40.2 (VSS), LED41.2 (VSS), LED42.2 (VSS), LED43.2 (VSS), LED44.2 (VSS), LED45.2 (VSS), LED46.2 (VSS), LED47.2 (VSS), LED48.2 (VSS), LED49.2 (VSS), LED5.2 (VSS), LED50.2 (VSS), LED51.2 (VSS), LED52.2 (VSS), LED53.2 (VSS), LED54.2 (VSS), LED55.2 (VSS), LED56.2 (VSS), LED57.2 (VSS), LED58.2 (VSS), LED59.2 (VSS), LED6.2 (VSS), LED60.2 (VSS), LED61.2 (VSS), LED62.2 (VSS), LED63.2 (VSS), LED64.2 (VSS), LED65.2 (VSS), LED66.2 (VSS), LED67.2 (VSS), LED68.2 (VSS), LED69.2 (VSS), LED7.2 (VSS), LED70.2 (VSS), LED71.2 (VSS), LED72.2 (VSS), LED73.2 (VSS), LED74.2 (VSS), LED75.2 (VSS), LED76.2 (VSS), LED77.2 (VSS), LED78.2 (VSS), LED79.2 (VSS), LED8.2 (VSS), LED80.2 (VSS), LED81.2 (VSS), LED82.2 (VSS), LED83.2 (VSS), LED84.2 (VSS), LED85.2 (VSS), LED86.2 (VSS), LED87.2 (VSS), LED88.2 (VSS), LED89.2 (VSS), LED9.2 (VSS), LED90.2 (VSS), LED91.2 (VSS), LED92.2 (VSS), LED93.2 (VSS), LED94.2 (VSS), LED95.2 (VSS), LED96.2 (VSS), LED97.2 (VSS), LED98.2 (VSS), LED99.2 (VSS)
- net at R4.2: now also LED1.4 (DIN); no longer LED1.3 (DIN)
- new net: LED17.2 (DOUT), LED18.4 (DIN)
- new net: LED16.2 (DOUT), LED17.4 (DIN)
- new net: LED54.2 (DOUT), LED55.4 (DIN)
- new net: LED87.2 (DOUT), LED88.4 (DIN)
- new net: LED6.2 (DOUT), LED7.4 (DIN)
- new net: LED5.2 (DOUT), LED6.4 (DIN)
- new net: LED75.2 (DOUT), LED76.4 (DIN)
- new net: LED74.2 (DOUT), LED75.4 (DIN)
- new net: LED78.2 (DOUT), LED79.4 (DIN)
- new net: LED77.2 (DOUT), LED78.4 (DIN)
- new net: LED36.2 (DOUT), LED37.4 (DIN)
- new net: LED35.2 (DOUT), LED36.4 (DIN)
- new net: LED62.2 (DOUT), LED63.4 (DIN)
- new net: LED61.2 (DOUT), LED62.4 (DIN)
- new net: LED59.2 (DOUT), LED60.4 (DIN)
- new net: LED58.2 (DOUT), LED59.4 (DIN)
- new net: LED47.2 (DOUT), LED48.4 (DIN)
- new net: LED46.2 (DOUT), LED47.4 (DIN)
- new net: LED92.2 (DOUT), LED93.4 (DIN)
- new net: LED91.2 (DOUT), LED92.4 (DIN)
- new net: LED21.2 (DOUT), LED22.4 (DIN)
- new net: LED20.2 (DOUT), LED21.4 (DIN)
- new net: LED23.2 (DOUT), LED24.4 (DIN)
- new net: LED22.2 (DOUT), LED23.4 (DIN)
- new net: LED28.2 (DOUT), LED29.4 (DIN)
- new net: LED27.2 (DOUT), LED28.4 (DIN)
- new net: LED51.2 (DOUT), LED52.4 (DIN)
- new net: LED50.2 (DOUT), LED51.4 (DIN)
- new net: LED10.2 (DOUT), LED11.4 (DIN)
- new net: LED10.4 (DIN), LED9.2 (DOUT)
- new net: LED39.2 (DOUT), LED40.4 (DIN)
- new net: LED38.2 (DOUT), LED39.4 (DIN)
- new net: LED31.2 (DOUT), LED32.4 (DIN)
- new net: LED30.2 (DOUT), LED31.4 (DIN)
- new net: LED82.2 (DOUT), LED83.4 (DIN)
- new net: LED81.2 (DOUT), LED82.4 (DIN)
- new net: LED19.2 (DOUT), LED20.4 (DIN)
- new net: LED18.2 (DOUT), LED19.4 (DIN)
- new net: DisplayLED1.4 (DIN), LED13.2 (DOUT)
- new net: LED12.2 (DOUT), LED13.4 (DIN)
- new net: LED100.4 (DIN), LED99.2 (DOUT)
- new net: LED98.2 (DOUT), LED99.4 (DIN)
- new net: LED53.2 (DOUT), LED54.4 (DIN)
- new net: LED52.2 (DOUT), LED53.4 (DIN)
- new net: LED73.2 (DOUT), LED74.4 (DIN)
- new net: LED72.2 (DOUT), LED73.4 (DIN)
- new net: LED90.2 (DOUT), LED91.4 (DIN)
- new net: LED89.2 (DOUT), LED90.4 (DIN)
- new net: LED41.2 (DOUT), LED42.4 (DIN)
- new net: LED40.2 (DOUT), LED41.4 (DIN)
- new net: LED86.2 (DOUT), LED87.4 (DIN)
- new net: LED68.2 (DOUT), LED69.4 (DIN)
- new net: LED67.2 (DOUT), LED68.4 (DIN)
- new net: LED4.2 (DOUT), LED5.4 (DIN)
- new net: DisplayLED1.2 (DOUT), DisplayLED2.4 (DIN)
- new net: LED37.2 (DOUT), LED38.4 (DIN)
- new net: LED48.2 (DOUT), LED49.4 (DIN)
- new net: LED15.2 (DOUT), LED16.4 (DIN)
- new net: LED79.2 (DOUT), LED80.4 (DIN)
- new net: LED49.2 (DOUT), LED50.4 (DIN)
- new net: LED33.2 (DOUT), LED34.4 (DIN)
- new net: LED11.2 (DOUT), LED12.4 (DIN)
- new net: LED93.2 (DOUT), LED94.4 (DIN)
- new net: LED97.2 (DOUT), LED98.4 (DIN)
- new net: LED96.2 (DOUT), LED97.4 (DIN)
- new net: LED14.2 (DOUT), LED15.4 (DIN)
- new net: LED32.2 (DOUT), LED33.4 (DIN)
- new net: LED29.2 (DOUT), LED30.4 (DIN)
- new net: LED101.2 (DOUT), R5.1
- new net: LED100.2 (DOUT), LED101.4 (DIN)
- new net: LED85.2 (DOUT), LED86.4 (DIN)
- new net: LED84.2 (DOUT), LED85.4 (DIN)
- new net: LED66.2 (DOUT), LED67.4 (DIN)
- new net: LED65.2 (DOUT), LED66.4 (DIN)
- new net: LED80.2 (DOUT), LED81.4 (DIN)
- new net: LED70.2 (DOUT), LED71.4 (DIN)
- new net: LED24.2 (DOUT), LED25.4 (DIN)
- new net: LED94.2 (DOUT), LED95.4 (DIN)
- new net: LED76.2 (DOUT), LED77.4 (DIN)
- new net: LED83.2 (DOUT), LED84.4 (DIN)
- new net: LED26.2 (DOUT), LED27.4 (DIN)
- new net: LED25.2 (DOUT), LED26.4 (DIN)
- new net: LED69.2 (DOUT), LED70.4 (DIN)
- new net: LED3.2 (DOUT), LED4.4 (DIN)
- new net: LED95.2 (DOUT), LED96.4 (DIN)
- new net: LED2.2 (DOUT), LED3.4 (DIN)
- new net: LED1.2 (DOUT), LED2.4 (DIN)
- new net: LED57.2 (DOUT), LED58.4 (DIN)
- new net: LED56.2 (DOUT), LED57.4 (DIN)
- new net: DisplayLED2.2 (DOUT), DisplayLED3.4 (DIN)
- new net: LED7.2 (DOUT), LED8.4 (DIN)
- new net: LED8.2 (DOUT), LED9.4 (DIN)
- new net: LED45.2 (DOUT), LED46.4 (DIN)
- new net: LED44.2 (DOUT), LED45.4 (DIN)
- new net: LED64.2 (DOUT), LED65.4 (DIN)
- new net: LED63.2 (DOUT), LED64.4 (DIN)
- new net: LED43.2 (DOUT), LED44.4 (DIN)
- new net: LED42.2 (DOUT), LED43.4 (DIN)
- new net: LED60.2 (DOUT), LED61.4 (DIN)
