File: MacOS Keyboard/STM32F072CBT6/ScottoModules.kicad_pcb (KiCad board)
At the start: 4 copper layers, 436 parts, among them J1 USB_C, SW1 SW_Push, SW2 RotaryEncoder, U1 STM32F072CBTx, U2 74AHCT125, U3 XC6206, U4 USBLC6-2SC6

Commit message: :P
Parts:
- removed the R2 at (-54.0, 39.4)
- removed the R2 at (-48.1, 3.24)
- removed the R3 at (-44.5, 3.12)
- added LEDBULKCAP2: 100uF, ScottoKeebs_Components:Capacitor_0402, B.Cu at (67.4, 184.6)
- added LEDBULKCAP3: 100uF, ScottoKeebs_Components:Capacitor_0402, B.Cu at (71.8, 203.7)
- added LEDBULKCAP4: 100uF, ScottoKeebs_Components:Capacitor_0402, B.Cu at (74.5, 222.7)
- added LEDBULKCAP5: 100uF, ScottoKeebs_Components:Capacitor_0402, B.Cu at (76.8, 241.8)
- added LEDBULKCAP6: 100uF, ScottoKeebs_Components:Capacitor_0402, B.Cu at (69.3, 260.8)
- added LEDCAP74: 100nF, ScottoKeebs_Components:Capacitor_0402, B.Cu at (130.1, 235.3)
- added LEDCAP91: 100nF, ScottoKeebs_Components:Capacitor_0402, B.Cu at (118.2, 254.3)
- added R2: 5.1k, ScottoKeebs_Components:Resistor_0402, B.Cu at (360.1, 129.5)
- added R5: 500R, ScottoKeebs_Components:Resistor_0402, B.Cu at (466.5, 256.8)
- DisplayLED1, DisplayLED2, DisplayLED3: footprint LED_SMD:LED_SK6812MINI_PLCC4_3.5x3.5mm_P1.75mm -> ScottoKeebs_Components:LED_SK6812MINI; moved to B.Cu
- DisplayLEDCAP2: renamed from DisplayLEDCAP1; moved to B.Cu
- DisplayLEDCAP3: renamed from DisplayLEDCAP2; moved to B.Cu
- LED1, LED10, LED100, LED101, LED11, LED12, LED13, LED14, LED15, LED16, LED17, LED18, LED19, LED2, LED20, LED21, LED22, LED23, LED24, LED25, LED26, LED27, LED28, LED29, LED3, LED30, LED31, LED32, LED33, LED34, LED35, LED36, LED37, LED38, LED39, LED4, LED40, LED41, LED42, LED43, LED44, LED45, LED46, LED47, LED48, LED49, LED5, LED50, LED51, LED52, LED53, LED54, LED55, LED56, LED57, LED58, LED59, LED6, LED60, LED61, LED62, LED63, LED64, LED65, LED66, LED67, LED68, LED69, LED7, LED70, LED71, LED72, LED73, LED74, LED75, LED76, LED77, LED78, LED79, LED8, LED80, LED81, LED82, LED83, LED84, LED85, LED86, LED87, LED88, LED89, LED9, LED90, LED91, LED92, LED93, LED94, LED95, LED96, LED97, LED98, LED99: footprint LED_SMD:LED_SK6812MINI_PLCC4_3.5x3.5mm_P1.75mm -> ScottoKeebs_Components:LED_SK6812MINI
- LEDBULKCAP1, R3, U2: moved to B.Cu
- R4: value 330R -> 500R; moved to B.Cu
- moved DisplayLED3 662.3 mm to (445.4, 147.6)
- moved DisplayLED2 627.5 mm to (423.9, 147.6)
- moved DisplayLEDCAP3 615.8 mm to (448.0, 152.2), turned to -90 degrees
- moved DisplayLED1 598.3 mm to (402.5, 147.6)
- moved SW2 577.3 mm to (471.7, 145.1)
- moved DisplayLEDCAP2 574.1 mm to (405.3, 152.3), turned to -90 degrees
- moved DisplayLEDCAP1 525.8 mm to (426.6, 152.3), turned to -90 degrees
- moved C15 453.2 mm to (391.6, 143.4), turned to 180 degrees
- moved C14 452.0 mm to (391.6, 142.4), turned to 180 degrees
- moved C11 449.9 mm to (380.8, 147.6), turned to 90 degrees
- moved C12 449.2 mm to (379.8, 147.6), turned to 90 degrees
- moved C7 448.9 mm to (389.7, 141.3), turned to 0 degrees
- moved C10 445.6 mm to (389.7, 138.7), turned to 180 degrees
- moved U1 444.4 mm to (383.5, 141.4), turned to 180 degrees
- moved C13 439.1 mm to (386.3, 135.3), turned to -90 degrees
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- renumbered DisplayLEDCAP102 to DisplayLEDCAP1
Connections:
- net A15 renamed /A15
- D1 pad 1: A5 -> A14
- D10 pad 1: A5 -> A14
- D100 pad 1: A10 -> B5
- D101 pad 1: A10 -> B5
- D11 pad 1: A5 -> A14
- D12 pad 1: A5 -> A14
- D13 pad 1: A5 -> A14
- D14 pad 1: A6 -> B9
- D15 pad 1: A6 -> B9
- D16 pad 1: A6 -> B9
- D17 pad 1: A6 -> B9
- D18 pad 1: A6 -> B9
- D19 pad 1: A6 -> B9
- D2 pad 1: A5 -> A14
- D20 pad 1: A6 -> B9
- D21 pad 1: A6 -> B9
- D22 pad 1: A6 -> B9
- D23 pad 1: A6 -> B9
- D24 pad 1: A6 -> B9
- D25 pad 1: A6 -> B9
- D26 pad 1: A6 -> B9
- D27 pad 1: A6 -> B9
- D28 pad 1: A6 -> B9
- D29 pad 1: A6 -> B9
- D3 pad 1: A5 -> A14
- D30 pad 1: A6 -> B9
- D31 pad 1: A6 -> B9
- D32 pad 1: A6 -> B9
- D33 pad 1: A6 -> B9
- D34 pad 1: A6 -> B9
- D35 pad 1: A7 -> B8
- D36 pad 1: A7 -> B8
- D37 pad 1: A7 -> B8
- D38 pad 1: A7 -> B8
- D39 pad 1: A7 -> B8
- D4 pad 1: A5 -> A14
- D40 pad 1: A7 -> B8
- D41 pad 1: A7 -> B8
- D42 pad 1: A7 -> B8
- D43 pad 1: A7 -> B8
- D44 pad 1: A7 -> B8
- D45 pad 1: A7 -> B8
- D46 pad 1: A7 -> B8
- D47 pad 1: A7 -> B8
- D48 pad 1: A7 -> B8
- D49 pad 1: A7 -> B8
- D5 pad 1: A5 -> A14
- D50 pad 1: A7 -> B8
- D51 pad 1: A7 -> B8
- D52 pad 1: A7 -> B8
- D53 pad 1: A7 -> B8
- D54 pad 1: A7 -> B8
- D55 pad 1: A7 -> B8
- D56 pad 1: A8 -> B7
- D57 pad 1: A8 -> B7
- D58 pad 1: A8 -> B7
- D59 pad 1: A8 -> B7
- D6 pad 1: A5 -> A14
- D60 pad 1: A8 -> B7
- D61 pad 1: A8 -> B7
- D62 pad 1: A8 -> B7
- D63 pad 1: A8 -> B7
- D64 pad 1: A8 -> B7
- D65 pad 1: A8 -> B7
- D66 pad 1: A8 -> B7
- D67 pad 1: A8 -> B7
- D68 pad 1: A8 -> B7
- D69 pad 1: A8 -> B7
- D7 pad 1: A5 -> A14
- D70 pad 1: A8 -> B7
- D71 pad 1: A8 -> B7
- D72 pad 1: A9 -> B6
- D73 pad 1: A9 -> B6
- D74 pad 1: A9 -> B6
- D75 pad 1: A9 -> B6
- D76 pad 1: A9 -> B6
- D77 pad 1: A9 -> B6
- D78 pad 1: A9 -> B6
- D79 pad 1: A9 -> B6
- D8 pad 1: A5 -> A14
- D80 pad 1: A9 -> B6
- D81 pad 1: A9 -> B6
- D82 pad 1: A9 -> B6
- D83 pad 1: A9 -> B6
- D84 pad 1: A9 -> B6
- D85 pad 1: A9 -> B6
- D86 pad 1: A9 -> B6
- D87 pad 1: A9 -> B6
- D88 pad 1: A9 -> B6
- D89 pad 1: A10 -> B5
- D9 pad 1: A5 -> A14
- D90 pad 1: A10 -> B5
- D91 pad 1: A10 -> B5
- D92 pad 1: A10 -> B5
- D93 pad 1: A10 -> B5
- D94 pad 1: A10 -> B5
- D95 pad 1: A10 -> B5
- D96 pad 1: A10 -> B5
- D97 pad 1: A10 -> B5
- D98 pad 1: A10 -> B5
- D99 pad 1: A10 -> B5
- DisplayLED1 pad 1: Net-(DisplayLED1-DOUT) -> +5V
- DisplayLED1 pad 2: GND -> Net-(DisplayLED1-DOUT)
- DisplayLED1 pad 3: Net-(DisplayLED1-DIN) -> GND
- DisplayLED1 pad 4: +5V -> Net-(DisplayLED1-DIN)
- DisplayLED2 pad 1: Net-(DisplayLED2-DOUT) -> +5V
- DisplayLED2 pad 2: GND -> Net-(DisplayLED2-DOUT)
- DisplayLED2 pad 3: Net-(DisplayLED1-DOUT) -> GND
- DisplayLED2 pad 4: +5V -> Net-(DisplayLED1-DOUT)
- DisplayLED3 pad 1: D1 -> +5V
- DisplayLED3 pad 2: GND -> D1
- DisplayLED3 pad 3: Net-(DisplayLED2-DOUT) -> GND
- DisplayLED3 pad 4: +5V -> Net-(DisplayLED2-DOUT)
- LED1 pad 1: Net-(LED1-DOUT) -> +5V
- LED1 pad 2: GND -> Net-(LED1-DOUT)
- LED1 pad 3: Net-(LED1-DIN) -> GND
- LED1 pad 4: +5V -> Net-(LED1-DIN)
- LED10 pad 1: Net-(LED10-DOUT) -> +5V
- LED10 pad 2: GND -> Net-(LED10-DOUT)
- LED10 pad 3: Net-(LED10-DIN) -> GND
- LED10 pad 4: +5V -> Net-(LED10-DIN)
- LED100 pad 1: Net-(LED100-DOUT) -> +5V
- LED100 pad 2: GND -> Net-(LED100-DOUT)
- LED100 pad 3: Net-(LED100-DIN) -> GND
- LED100 pad 4: +5V -> Net-(LED100-DIN)
- LED101 pad 1: unconnected-(LED101-DOUT-Pad1) -> +5V
- LED101 pad 2: GND -> Net-(LED101-DOUT)
- LED101 pad 3: Net-(LED100-DOUT) -> GND
- LED101 pad 4: +5V -> Net-(LED100-DOUT)
- LED11 pad 1: Net-(LED11-DOUT) -> +5V
- LED11 pad 2: GND -> Net-(LED11-DOUT)
- LED11 pad 3: Net-(LED10-DOUT) -> GND
- LED11 pad 4: +5V -> Net-(LED10-DOUT)
- LED12 pad 1: Net-(LED12-DOUT) -> +5V
- LED12 pad 2: GND -> Net-(LED12-DOUT)
- LED12 pad 3: Net-(LED11-DOUT) -> GND
- LED12 pad 4: +5V -> Net-(LED11-DOUT)
- LED13 pad 1: Net-(DisplayLED1-DIN) -> +5V
- LED13 pad 2: GND -> Net-(DisplayLED1-DIN)
- LED13 pad 3: Net-(LED12-DOUT) -> GND
- LED13 pad 4: +5V -> Net-(LED12-DOUT)
- LED14 pad 1: Net-(LED14-DOUT) -> +5V
- LED14 pad 2: GND -> Net-(LED14-DOUT)
- LED14 pad 3: D1 -> GND
- LED14 pad 4: +5V -> D1
- LED15 pad 1: Net-(LED15-DOUT) -> +5V
- LED15 pad 2: GND -> Net-(LED15-DOUT)
- LED15 pad 3: Net-(LED14-DOUT) -> GND
- LED15 pad 4: +5V -> Net-(LED14-DOUT)
- LED16 pad 1: Net-(LED16-DOUT) -> +5V
- LED16 pad 2: GND -> Net-(LED16-DOUT)
- LED16 pad 3: Net-(LED15-DOUT) -> GND
- LED16 pad 4: +5V -> Net-(LED15-DOUT)
- LED17 pad 1: Net-(LED17-DOUT) -> +5V
- LED17 pad 2: GND -> Net-(LED17-DOUT)
- LED17 pad 3: Net-(LED16-DOUT) -> GND
- LED17 pad 4: +5V -> Net-(LED16-DOUT)
- LED18 pad 1: Net-(LED18-DOUT) -> +5V
- LED18 pad 2: GND -> Net-(LED18-DOUT)
- LED18 pad 3: Net-(LED17-DOUT) -> GND
- LED18 pad 4: +5V -> Net-(LED17-DOUT)
- LED19 pad 1: Net-(LED19-DOUT) -> +5V
- LED19 pad 2: GND -> Net-(LED19-DOUT)
- LED19 pad 3: Net-(LED18-DOUT) -> GND
- LED19 pad 4: +5V -> Net-(LED18-DOUT)
- LED2 pad 1: Net-(LED2-DOUT) -> +5V
- LED2 pad 2: GND -> Net-(LED2-DOUT)
- LED2 pad 3: Net-(LED1-DOUT) -> GND
- LED2 pad 4: +5V -> Net-(LED1-DOUT)
- LED20 pad 1: Net-(LED20-DOUT) -> +5V
- LED20 pad 2: GND -> Net-(LED20-DOUT)
- LED20 pad 3: Net-(LED19-DOUT) -> GND
- LED20 pad 4: +5V -> Net-(LED19-DOUT)
- LED21 pad 1: Net-(LED21-DOUT) -> +5V
- LED21 pad 2: GND -> Net-(LED21-DOUT)
- LED21 pad 3: Net-(LED20-DOUT) -> GND
- LED21 pad 4: +5V -> Net-(LED20-DOUT)
- LED22 pad 1: Net-(LED22-DOUT) -> +5V
- LED22 pad 2: GND -> Net-(LED22-DOUT)
- LED22 pad 3: Net-(LED21-DOUT) -> GND
- LED22 pad 4: +5V -> Net-(LED21-DOUT)
- LED23 pad 1: Net-(LED23-DOUT) -> +5V
- LED23 pad 2: GND -> Net-(LED23-DOUT)
- LED23 pad 3: Net-(LED22-DOUT) -> GND
- LED23 pad 4: +5V -> Net-(LED22-DOUT)
- LED24 pad 1: Net-(LED24-DOUT) -> +5V
- LED24 pad 2: GND -> Net-(LED24-DOUT)
- LED24 pad 3: Net-(LED23-DOUT) -> GND
- LED24 pad 4: +5V -> Net-(LED23-DOUT)
- LED25 pad 1: Net-(LED25-DOUT) -> +5V
- LED25 pad 2: GND -> Net-(LED25-DOUT)
- LED25 pad 3: Net-(LED24-DOUT) -> GND
- LED25 pad 4: +5V -> Net-(LED24-DOUT)
- LED26 pad 1: Net-(LED26-DOUT) -> +5V
- LED26 pad 2: GND -> Net-(LED26-DOUT)
- LED26 pad 3: Net-(LED25-DOUT) -> GND
- LED26 pad 4: +5V -> Net-(LED25-DOUT)
- LED27 pad 1: Net-(LED27-DOUT) -> +5V
- LED27 pad 2: GND -> Net-(LED27-DOUT)
- LED27 pad 3: Net-(LED26-DOUT) -> GND
- LED27 pad 4: +5V -> Net-(LED26-DOUT)
- LED28 pad 1: Net-(LED28-DOUT) -> +5V
- LED28 pad 2: GND -> Net-(LED28-DOUT)
- LED28 pad 3: Net-(LED27-DOUT) -> GND
- LED28 pad 4: +5V -> Net-(LED27-DOUT)
- LED29 pad 1: Net-(LED29-DOUT) -> +5V
- LED29 pad 2: GND -> Net-(LED29-DOUT)
- LED29 pad 3: Net-(LED28-DOUT) -> GND
- LED29 pad 4: +5V -> Net-(LED28-DOUT)
- LED3 pad 1: Net-(LED3-DOUT) -> +5V
- LED3 pad 2: GND -> Net-(LED3-DOUT)
- LED3 pad 3: Net-(LED2-DOUT) -> GND
- LED3 pad 4: +5V -> Net-(LED2-DOUT)
- LED30 pad 1: Net-(LED30-DOUT) -> +5V
- LED30 pad 2: GND -> Net-(LED30-DOUT)
- LED30 pad 3: Net-(LED29-DOUT) -> GND
- LED30 pad 4: +5V -> Net-(LED29-DOUT)
- LED31 pad 1: Net-(LED31-DOUT) -> +5V
- LED31 pad 2: GND -> Net-(LED31-DOUT)
- LED31 pad 3: Net-(LED30-DOUT) -> GND
- LED31 pad 4: +5V -> Net-(LED30-DOUT)
- LED32 pad 1: Net-(LED32-DOUT) -> +5V
- LED32 pad 2: GND -> Net-(LED32-DOUT)
- LED32 pad 3: Net-(LED31-DOUT) -> GND
- LED32 pad 4: +5V -> Net-(LED31-DOUT)
- LED33 pad 1: Net-(LED33-DOUT) -> +5V
- LED33 pad 2: GND -> Net-(LED33-DOUT)
- LED33 pad 3: Net-(LED32-DOUT) -> GND
- LED33 pad 4: +5V -> Net-(LED32-DOUT)
- LED34 pad 1: D2 -> +5V
- LED34 pad 2: GND -> D2
- LED34 pad 3: Net-(LED33-DOUT) -> GND
- LED34 pad 4: +5V -> Net-(LED33-DOUT)
- LED35 pad 1: Net-(LED35-DOUT) -> +5V
- LED35 pad 2: GND -> Net-(LED35-DOUT)
- LED35 pad 3: D2 -> GND
- LED35 pad 4: +5V -> D2
- LED36 pad 1: Net-(LED36-DOUT) -> +5V
- LED36 pad 2: GND -> Net-(LED36-DOUT)
- LED36 pad 3: Net-(LED35-DOUT) -> GND
- LED36 pad 4: +5V -> Net-(LED35-DOUT)
- LED37 pad 1: Net-(LED37-DOUT) -> +5V
- LED37 pad 2: GND -> Net-(LED37-DOUT)
- LED37 pad 3: Net-(LED36-DOUT) -> GND
- LED37 pad 4: +5V -> Net-(LED36-DOUT)
- LED38 pad 1: Net-(LED38-DOUT) -> +5V
- LED38 pad 2: GND -> Net-(LED38-DOUT)
- LED38 pad 3: Net-(LED37-DOUT) -> GND
- LED38 pad 4: +5V -> Net-(LED37-DOUT)
- LED39 pad 1: Net-(LED39-DOUT) -> +5V
- LED39 pad 2: GND -> Net-(LED39-DOUT)
- LED39 pad 3: Net-(LED38-DOUT) -> GND
- LED39 pad 4: +5V -> Net-(LED38-DOUT)
- LED4 pad 1: Net-(LED4-DOUT) -> +5V
- LED4 pad 2: GND -> Net-(LED4-DOUT)
- LED4 pad 3: Net-(LED3-DOUT) -> GND
- LED4 pad 4: +5V -> Net-(LED3-DOUT)
- LED40 pad 1: Net-(LED40-DOUT) -> +5V
- LED40 pad 2: GND -> Net-(LED40-DOUT)
- LED40 pad 3: Net-(LED39-DOUT) -> GND
- LED40 pad 4: +5V -> Net-(LED39-DOUT)
- LED41 pad 1: Net-(LED41-DOUT) -> +5V
- LED41 pad 2: GND -> Net-(LED41-DOUT)
- LED41 pad 3: Net-(LED40-DOUT) -> GND
- LED41 pad 4: +5V -> Net-(LED40-DOUT)
- LED42 pad 1: Net-(LED42-DOUT) -> +5V
- LED42 pad 2: GND -> Net-(LED42-DOUT)
- LED42 pad 3: Net-(LED41-DOUT) -> GND
- LED42 pad 4: +5V -> Net-(LED41-DOUT)
- LED43 pad 1: Net-(LED43-DOUT) -> +5V
- LED43 pad 2: GND -> Net-(LED43-DOUT)
- LED43 pad 3: Net-(LED42-DOUT) -> GND
- LED43 pad 4: +5V -> Net-(LED42-DOUT)
- LED44 pad 1: Net-(LED44-DOUT) -> +5V
- LED44 pad 2: GND -> Net-(LED44-DOUT)
- LED44 pad 3: Net-(LED43-DOUT) -> GND
- LED44 pad 4: +5V -> Net-(LED43-DOUT)
- LED45 pad 1: Net-(LED45-DOUT) -> +5V
- LED45 pad 2: GND -> Net-(LED45-DOUT)
- LED45 pad 3: Net-(LED44-DOUT) -> GND
- LED45 pad 4: +5V -> Net-(LED44-DOUT)
- LED46 pad 1: Net-(LED46-DOUT) -> +5V
- LED46 pad 2: GND -> Net-(LED46-DOUT)
- LED46 pad 3: Net-(LED45-DOUT) -> GND
- LED46 pad 4: +5V -> Net-(LED45-DOUT)
- LED47 pad 1: Net-(LED47-DOUT) -> +5V
- LED47 pad 2: GND -> Net-(LED47-DOUT)
- LED47 pad 3: Net-(LED46-DOUT) -> GND
- LED47 pad 4: +5V -> Net-(LED46-DOUT)
- LED48 pad 1: Net-(LED48-DOUT) -> +5V
- LED48 pad 2: GND -> Net-(LED48-DOUT)
- LED48 pad 3: Net-(LED47-DOUT) -> GND
- LED48 pad 4: +5V -> Net-(LED47-DOUT)
- LED49 pad 1: Net-(LED49-DOUT) -> +5V
- LED49 pad 2: GND -> Net-(LED49-DOUT)
- LED49 pad 3: Net-(LED48-DOUT) -> GND
- LED49 pad 4: +5V -> Net-(LED48-DOUT)
- LED5 pad 1: Net-(LED5-DOUT) -> +5V
- LED5 pad 2: GND -> Net-(LED5-DOUT)
- LED5 pad 3: Net-(LED4-DOUT) -> GND
- LED5 pad 4: +5V -> Net-(LED4-DOUT)
- LED50 pad 1: Net-(LED50-DOUT) -> +5V
- LED50 pad 2: GND -> Net-(LED50-DOUT)
- LED50 pad 3: Net-(LED49-DOUT) -> GND
- LED50 pad 4: +5V -> Net-(LED49-DOUT)
- LED51 pad 1: Net-(LED51-DOUT) -> +5V
- LED51 pad 2: GND -> Net-(LED51-DOUT)
- LED51 pad 3: Net-(LED50-DOUT) -> GND
- LED51 pad 4: +5V -> Net-(LED50-DOUT)
- LED52 pad 1: Net-(LED52-DOUT) -> +5V
- LED52 pad 2: GND -> Net-(LED52-DOUT)
- LED52 pad 3: Net-(LED51-DOUT) -> GND
- LED52 pad 4: +5V -> Net-(LED51-DOUT)
- LED53 pad 1: Net-(LED53-DOUT) -> +5V
- LED53 pad 2: GND -> Net-(LED53-DOUT)
- LED53 pad 3: Net-(LED52-DOUT) -> GND
- LED53 pad 4: +5V -> Net-(LED52-DOUT)
- LED54 pad 1: Net-(LED54-DOUT) -> +5V
- LED54 pad 2: GND -> Net-(LED54-DOUT)
- LED54 pad 3: Net-(LED53-DOUT) -> GND
- LED54 pad 4: +5V -> Net-(LED53-DOUT)
- LED55 pad 1: D3 -> +5V
- LED55 pad 2: GND -> D3
- LED55 pad 3: Net-(LED54-DOUT) -> GND
- LED55 pad 4: +5V -> Net-(LED54-DOUT)
- LED56 pad 1: Net-(LED56-DOUT) -> +5V
- LED56 pad 2: GND -> Net-(LED56-DOUT)
- LED56 pad 3: D3 -> GND
- LED56 pad 4: +5V -> D3
- LED57 pad 1: Net-(LED57-DOUT) -> +5V
- LED57 pad 2: GND -> Net-(LED57-DOUT)
- LED57 pad 3: Net-(LED56-DOUT) -> GND
- LED57 pad 4: +5V -> Net-(LED56-DOUT)
- LED58 pad 1: Net-(LED58-DOUT) -> +5V
- LED58 pad 2: GND -> Net-(LED58-DOUT)
- LED58 pad 3: Net-(LED57-DOUT) -> GND
- LED58 pad 4: +5V -> Net-(LED57-DOUT)
- LED59 pad 1: Net-(LED59-DOUT) -> +5V
- LED59 pad 2: GND -> Net-(LED59-DOUT)
- LED59 pad 3: Net-(LED58-DOUT) -> GND
- LED59 pad 4: +5V -> Net-(LED58-DOUT)
- LED6 pad 1: Net-(LED6-DOUT) -> +5V
- LED6 pad 2: GND -> Net-(LED6-DOUT)
- LED6 pad 3: Net-(LED5-DOUT) -> GND
- LED6 pad 4: +5V -> Net-(LED5-DOUT)
- LED60 pad 1: Net-(LED60-DOUT) -> +5V
- LED60 pad 2: GND -> Net-(LED60-DOUT)
- LED60 pad 3: Net-(LED59-DOUT) -> GND
- LED60 pad 4: +5V -> Net-(LED59-DOUT)
- LED61 pad 1: Net-(LED61-DOUT) -> +5V
- LED61 pad 2: GND -> Net-(LED61-DOUT)
- LED61 pad 3: Net-(LED60-DOUT) -> GND
- LED61 pad 4: +5V -> Net-(LED60-DOUT)
- LED62 pad 1: Net-(LED62-DOUT) -> +5V
- LED62 pad 2: GND -> Net-(LED62-DOUT)
- LED62 pad 3: Net-(LED61-DOUT) -> GND
- LED62 pad 4: +5V -> Net-(LED61-DOUT)
- LED63 pad 1: Net-(LED63-DOUT) -> +5V
- LED63 pad 2: GND -> Net-(LED63-DOUT)
- LED63 pad 3: Net-(LED62-DOUT) -> GND
- LED63 pad 4: +5V -> Net-(LED62-DOUT)
- LED64 pad 1: Net-(LED64-DOUT) -> +5V
- LED64 pad 2: GND -> Net-(LED64-DOUT)
- LED64 pad 3: Net-(LED63-DOUT) -> GND
- LED64 pad 4: +5V -> Net-(LED63-DOUT)
- LED65 pad 1: Net-(LED65-DOUT) -> +5V
- LED65 pad 2: GND -> Net-(LED65-DOUT)
- LED65 pad 3: Net-(LED64-DOUT) -> GND
- LED65 pad 4: +5V -> Net-(LED64-DOUT)
- LED66 pad 1: Net-(LED66-DOUT) -> +5V
- LED66 pad 2: GND -> Net-(LED66-DOUT)
- LED66 pad 3: Net-(LED65-DOUT) -> GND
- LED66 pad 4: +5V -> Net-(LED65-DOUT)
- LED67 pad 1: Net-(LED67-DOUT) -> +5V
- LED67 pad 2: GND -> Net-(LED67-DOUT)
- LED67 pad 3: Net-(LED66-DOUT) -> GND
- LED67 pad 4: +5V -> Net-(LED66-DOUT)
- LED68 pad 1: Net-(LED68-DOUT) -> +5V
- LED68 pad 2: GND -> Net-(LED68-DOUT)
- LED68 pad 3: Net-(LED67-DOUT) -> GND
- LED68 pad 4: +5V -> Net-(LED67-DOUT)
- LED69 pad 1: Net-(LED69-DOUT) -> +5V
- LED69 pad 2: GND -> Net-(LED69-DOUT)
- LED69 pad 3: Net-(LED68-DOUT) -> GND
- LED69 pad 4: +5V -> Net-(LED68-DOUT)
- LED7 pad 1: Net-(LED7-DOUT) -> +5V
- LED7 pad 2: GND -> Net-(LED7-DOUT)
- LED7 pad 3: Net-(LED6-DOUT) -> GND
- LED7 pad 4: +5V -> Net-(LED6-DOUT)
- LED70 pad 1: Net-(LED70-DOUT) -> +5V
- LED70 pad 2: GND -> Net-(LED70-DOUT)
- LED70 pad 3: Net-(LED69-DOUT) -> GND
- LED70 pad 4: +5V -> Net-(LED69-DOUT)
- LED71 pad 1: D4 -> +5V
- LED71 pad 2: GND -> D4
- LED71 pad 3: Net-(LED70-DOUT) -> GND
- LED71 pad 4: +5V -> Net-(LED70-DOUT)
- LED72 pad 1: Net-(LED72-DOUT) -> +5V
- LED72 pad 2: GND -> Net-(LED72-DOUT)
- LED72 pad 3: D4 -> GND
- LED72 pad 4: +5V -> D4
- LED73 pad 1: Net-(LED73-DOUT) -> +5V
- LED73 pad 2: GND -> Net-(LED73-DOUT)
- LED73 pad 3: Net-(LED72-DOUT) -> GND
- LED73 pad 4: +5V -> Net-(LED72-DOUT)
- LED74 pad 1: Net-(LED74-DOUT) -> +5V
- LED74 pad 2: GND -> Net-(LED74-DOUT)
- LED74 pad 3: Net-(LED73-DOUT) -> GND
- LED74 pad 4: +5V -> Net-(LED73-DOUT)
- LED75 pad 1: Net-(LED75-DOUT) -> +5V
- LED75 pad 2: GND -> Net-(LED75-DOUT)
- LED75 pad 3: Net-(LED74-DOUT) -> GND
- LED75 pad 4: +5V -> Net-(LED74-DOUT)
- LED76 pad 1: Net-(LED76-DOUT) -> +5V
- LED76 pad 2: GND -> Net-(LED76-DOUT)
- LED76 pad 3: Net-(LED75-DOUT) -> GND
- LED76 pad 4: +5V -> Net-(LED75-DOUT)
- LED77 pad 1: Net-(LED77-DOUT) -> +5V
- LED77 pad 2: GND -> Net-(LED77-DOUT)
- LED77 pad 3: Net-(LED76-DOUT) -> GND
- LED77 pad 4: +5V -> Net-(LED76-DOUT)
- LED78 pad 1: Net-(LED78-DOUT) -> +5V
- LED78 pad 2: GND -> Net-(LED78-DOUT)
- LED78 pad 3: Net-(LED77-DOUT) -> GND
- LED78 pad 4: +5V -> Net-(LED77-DOUT)
- LED79 pad 1: Net-(LED79-DOUT) -> +5V
- LED79 pad 2: GND -> Net-(LED79-DOUT)
- LED79 pad 3: Net-(LED78-DOUT) -> GND
- LED79 pad 4: +5V -> Net-(LED78-DOUT)
- LED8 pad 1: Net-(LED8-DOUT) -> +5V
- LED8 pad 2: GND -> Net-(LED8-DOUT)
- LED8 pad 3: Net-(LED7-DOUT) -> GND
- LED8 pad 4: +5V -> Net-(LED7-DOUT)
- LED80 pad 1: Net-(LED80-DOUT) -> +5V
- LED80 pad 2: GND -> Net-(LED80-DOUT)
- LED80 pad 3: Net-(LED79-DOUT) -> GND
- LED80 pad 4: +5V -> Net-(LED79-DOUT)
- LED81 pad 1: Net-(LED81-DOUT) -> +5V
- LED81 pad 2: GND -> Net-(LED81-DOUT)
- LED81 pad 3: Net-(LED80-DOUT) -> GND
- LED81 pad 4: +5V -> Net-(LED80-DOUT)
- LED82 pad 1: Net-(LED82-DOUT) -> +5V
- LED82 pad 2: GND -> Net-(LED82-DOUT)
- LED82 pad 3: Net-(LED81-DOUT) -> GND
- LED82 pad 4: +5V -> Net-(LED81-DOUT)
- LED83 pad 1: Net-(LED83-DOUT) -> +5V
- LED83 pad 2: GND -> Net-(LED83-DOUT)
- LED83 pad 3: Net-(LED82-DOUT) -> GND
- LED83 pad 4: +5V -> Net-(LED82-DOUT)
- LED84 pad 1: Net-(LED84-DOUT) -> +5V
- LED84 pad 2: GND -> Net-(LED84-DOUT)
- LED84 pad 3: Net-(LED83-DOUT) -> GND
- LED84 pad 4: +5V -> Net-(LED83-DOUT)
- LED85 pad 1: Net-(LED85-DOUT) -> +5V
- LED85 pad 2: GND -> Net-(LED85-DOUT)
- LED85 pad 3: Net-(LED84-DOUT) -> GND
- LED85 pad 4: +5V -> Net-(LED84-DOUT)
- LED86 pad 1: Net-(LED86-DOUT) -> +5V
- LED86 pad 2: GND -> Net-(LED86-DOUT)
- LED86 pad 3: Net-(LED85-DOUT) -> GND
- LED86 pad 4: +5V -> Net-(LED85-DOUT)
- LED87 pad 1: Net-(LED87-DOUT) -> +5V
- LED87 pad 2: GND -> Net-(LED87-DOUT)
- LED87 pad 3: Net-(LED86-DOUT) -> GND
- LED87 pad 4: +5V -> Net-(LED86-DOUT)
- LED88 pad 1: D5 -> +5V
- LED88 pad 2: GND -> D5
- LED88 pad 3: Net-(LED87-DOUT) -> GND
- LED88 pad 4: +5V -> Net-(LED87-DOUT)
- LED89 pad 1: Net-(LED89-DOUT) -> +5V
- LED89 pad 2: GND -> Net-(LED89-DOUT)
- LED89 pad 3: D5 -> GND
- LED89 pad 4: +5V -> D5
- LED9 pad 1: Net-(LED10-DIN) -> +5V
- LED9 pad 2: GND -> Net-(LED10-DIN)
- LED9 pad 3: Net-(LED8-DOUT) -> GND
- LED9 pad 4: +5V -> Net-(LED8-DOUT)
- LED90 pad 1: Net-(LED90-DOUT) -> +5V
- LED90 pad 2: GND -> Net-(LED90-DOUT)
- LED90 pad 3: Net-(LED89-DOUT) -> GND
- LED90 pad 4: +5V -> Net-(LED89-DOUT)
- LED91 pad 1: Net-(LED91-DOUT) -> +5V
- LED91 pad 2: GND -> Net-(LED91-DOUT)
- LED91 pad 3: Net-(LED90-DOUT) -> GND
- LED91 pad 4: +5V -> Net-(LED90-DOUT)
- LED92 pad 1: Net-(LED92-DOUT) -> +5V
- LED92 pad 2: GND -> Net-(LED92-DOUT)
- LED92 pad 3: Net-(LED91-DOUT) -> GND
- LED92 pad 4: +5V -> Net-(LED91-DOUT)
- LED93 pad 1: Net-(LED93-DOUT) -> +5V
- LED93 pad 2: GND -> Net-(LED93-DOUT)
- LED93 pad 3: Net-(LED92-DOUT) -> GND
- LED93 pad 4: +5V -> Net-(LED92-DOUT)
- LED94 pad 1: Net-(LED94-DOUT) -> +5V
- LED94 pad 2: GND -> Net-(LED94-DOUT)
- LED94 pad 3: Net-(LED93-DOUT) -> GND
- LED94 pad 4: +5V -> Net-(LED93-DOUT)
- LED95 pad 1: Net-(LED95-DOUT) -> +5V
- LED95 pad 2: GND -> Net-(LED95-DOUT)
- LED95 pad 3: Net-(LED94-DOUT) -> GND
- LED95 pad 4: +5V -> Net-(LED94-DOUT)
- LED96 pad 1: Net-(LED96-DOUT) -> +5V
- LED96 pad 2: GND -> Net-(LED96-DOUT)
- LED96 pad 3: Net-(LED95-DOUT) -> GND
- LED96 pad 4: +5V -> Net-(LED95-DOUT)
- LED97 pad 1: Net-(LED97-DOUT) -> +5V
- LED97 pad 2: GND -> Net-(LED97-DOUT)
- LED97 pad 3: Net-(LED96-DOUT) -> GND
- LED97 pad 4: +5V -> Net-(LED96-DOUT)
- LED98 pad 1: Net-(LED98-DOUT) -> +5V
- LED98 pad 2: GND -> Net-(LED98-DOUT)
- LED98 pad 3: Net-(LED97-DOUT) -> GND
- LED98 pad 4: +5V -> Net-(LED97-DOUT)
- LED99 pad 1: Net-(LED100-DIN) -> +5V
- LED99 pad 2: GND -> Net-(LED100-DIN)
- LED99 pad 3: Net-(LED98-DOUT) -> GND
- LED99 pad 4: +5V -> Net-(LED98-DOUT)
- S1 pad 1: B0 -> A13
- S10 pad 1: B9 -> B10
- S100 pad 1: A1 -> A3
- S101 pad 1: A3 -> A1
- S11 pad 1: B10 -> B2
- S12 pad 1: B11 -> B1
- S13 pad 1: B12 -> B0
- S14 pad 1: B0 -> A13
- S15 pad 1: B1 -> A10
- S16 pad 1: B2 -> A9
- S17 pad 1: B3 -> A8
- S18 pad 1: B4 -> B15
- S19 pad 1: B5 -> B14
- S2 pad 1: B1 -> A10
- S20 pad 1: B6 -> B13
- S21 pad 1: B7 -> B12
- S22 pad 1: B8 -> B11
- S23 pad 1: B9 -> B10
- S24 pad 1: B10 -> B2
- S25 pad 1: B11 -> B1
- S26 pad 1: B12 -> B0
- S27 pad 1: B13 -> A7
- S28 pad 1: B14 -> A6
- S29 pad 1: B15 -> A5
- S3 pad 1: B2 -> A9
- S30 pad 1: A13 -> A4
- S31 pad 1: A1 -> A3
- S33 pad 1: A3 -> A1
- S34 pad 1: A4 -> A0
- S35 pad 1: B0 -> A13
- S36 pad 1: B1 -> A10
- S37 pad 1: B2 -> A9
- S38 pad 1: B3 -> A8
- S39 pad 1: B4 -> B15
- S4 pad 1: B3 -> A8
- S40 pad 1: B5 -> B14
- S41 pad 1: B6 -> B13
- S42 pad 1: B7 -> B12
- S43 pad 1: B8 -> B11
- S44 pad 1: B9 -> B10
- S45 pad 1: B10 -> B2
- S46 pad 1: B11 -> B1
- S47 pad 1: B12 -> B0
- S48 pad 1: B13 -> A7
- S49 pad 1: B14 -> A6
- S5 pad 1: B4 -> B15
- S50 pad 1: B15 -> A5
- S51 pad 1: A13 -> A4
- S52 pad 1: A1 -> A3
- S54 pad 1: A3 -> A1
- S55 pad 1: A4 -> A0
- S56 pad 1: B0 -> A13
- S57 pad 1: B1 -> A10
- S58 pad 1: B2 -> A9
- S59 pad 1: B3 -> A8
- S6 pad 1: B5 -> B14
- S60 pad 1: B4 -> B15
- S61 pad 1: B5 -> B14
- S62 pad 1: B6 -> B13
- S63 pad 1: B7 -> B12
- S64 pad 1: B8 -> B11
- S65 pad 1: B9 -> B10
- S66 pad 1: B10 -> B2
- S67 pad 1: B11 -> B1
- S68 pad 1: B13 -> A7
- S69 pad 1: A1 -> A3
- S7 pad 1: B6 -> B13
- S71 pad 1: A3 -> A1
- S72 pad 1: B0 -> A13
- S73 pad 1: B2 -> A9
- S74 pad 1: B3 -> A8
- S75 pad 1: B4 -> B15
- S76 pad 1: B5 -> B14
- S77 pad 1: B6 -> B13
- S78 pad 1: B7 -> B12
- S79 pad 1: B8 -> B11
- S8 pad 1: B7 -> B12
- S80 pad 1: B9 -> B10
- S81 pad 1: B10 -> B2
- S82 pad 1: B11 -> B1
- S83 pad 1: B13 -> A7
- S84 pad 1: B15 -> A5
- S85 pad 1: A1 -> A3
- S87 pad 1: A3 -> A1
- S88 pad 1: A4 -> A0
- S89 pad 1: B0 -> A13
- S9 pad 1: B8 -> B11
- S90 pad 1: B2 -> A9
- S91 pad 1: B3 -> A8
- S92 pad 1: B6 -> B13
- S93 pad 1: B10 -> B2
- S94 pad 1: B11 -> B1
- S95 pad 1: B12 -> B0
- S96 pad 1: B13 -> A7
- S97 pad 1: B14 -> A6
- S98 pad 1: B15 -> A5
- S99 pad 1: A13 -> A4
- SW2 pad A: /A0 -> /B3
- SW2 pad B: /A14 -> /B4
- U1 pad 10: /A0 -> A0
- U1 pad 37: /A14 -> A14
- U1 pad 39: B3 -> /B3
- U1 pad 40: B4 -> /B4
Routing:
- net GND: track 47810.3 -> 306.6 mm, vias 0 -> 30
- net +5V: track 30.5 -> 3148.7 mm, vias 0 -> 161
- net B5: track 107.4 -> 638.5 mm
- net B7: track 107.4 -> 598.2 mm, vias 0 -> 2
- net D1: track 0.00 -> 481.9 mm, vias 0 -> 2
- net B6: track 127.5 -> 609.3 mm
- net B8: track 107.4 -> 579.1 mm
- net D3: track 0.00 -> 449.3 mm, vias 0 -> 2
- net D2: track 0.00 -> 435.9 mm, vias 0 -> 2
- net D5: track 0.00 -> 434.6 mm, vias 0 -> 2
- net B9: track 116.9 -> 536.0 mm
- net D4: track 0.00 -> 408.1 mm, vias 0 -> 2
- net A9: track 0.00 -> 403.3 mm
- net A8: track 0.00 -> 382.7 mm
- net A10: track 0.00 -> 373.7 mm
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- added copper zone on B.Cu, net GND
- added copper zone on F.Cu, net GND
Other:
- board outline added: 439.4 x 157.7 mm
