File: MacOS Keyboard/STM32F072CBT6/ScottoModules.kicad_pcb (KiCad board)
At the start: 4 copper layers, 439.4 x 157.7 mm, 442 parts, among them J1 USB_C, SW1 SW_Push, SW2 RotaryEncoder, U1 STM32F072CBTx, U2 74AHCT125, U3 XC6206, U4 USBLC6-2SC6

Commit message: asdasda
Parts:
- removed the LEDCAP74 at (130.1, 235.3)
- removed the LEDCAP91 at (118.2, 254.3)
Routing:
- net GND: track 306.6 -> 328.9 mm, vias 30 -> 105
- net +5V: track 3148.7 -> 3138.2 mm, vias 161 -> 159
- net +3.3V: track 92.9 -> 91.8 mm
- net /B3: vias 2 -> 1
Other:
- copper layers 4 -> 2
