File: MacOS Keyboard/STM32F072CBT6/ScottoModules.kicad_sch (KiCad schematic)
At the start: 224 parts, among them J1 USB_C, SW1 SW_Push, U1 74AHCT125, U2 STM32F072CBTx, U3 XC6206, U4 USBLC6-2SC6

Commit message: things
Parts:
- removed RV1: R_Potentiometer, Potentiometer_THT:Potentiometer_Bourns_3266W_Vertical, symbol Device:R_Potentiometer
- removed U1: 74AHCT125, Package_DIP:DIP-14_W7.62mm, symbol 74xx:74AHCT125
- removed U2: STM32F072CBTx, Package_QFP:LQFP-48_7x7mm_P0.5mm, symbol MCU_ST_STM32F0:STM32F072CBTx
- added SW2: RotaryEncoder, Rotary_Encoder:RotaryEncoder_Alps_EC11E_Vertical_H20mm, symbol Device:RotaryEncoder
- added U1: STM32F072CBTx, Package_QFP:LQFP-48_7x7mm_P0.5mm, symbol MCU_ST_STM32F0:STM32F072CBTx
- added U2: 74AHCT125, Package_DIP:DIP-14_W7.62mm, symbol 74xx:74AHCT125
- R1: LCSC (none) -> C25744
Connections:
- net +3.3V: now also U1.1 (VBAT), U1.24 (VDD), U1.36 (VDDIO2), U1.48 (VDD), U1.9 (VDDA)
- net +5V: now also U2.14 (VCC)
- net A0: now also SW2.A, U1.10 (PA0)
- net A1: now also U1.11 (PA1)
- net A10: now also U1.31 (PA10)
- net A13: now also U1.34 (PA13)
- net A14: now also SW2.B, U1.37 (PA14)
- net A15: now also U1.38 (PA15), U2.2
- net A2: now also U1.12 (PA2)
- net A3: now also U1.13 (PA3)
- net A4: now also U1.14 (PA4)
- net A5: now also U1.15 (PA5)
- net A6: now also U1.16 (PA6)
- net A7: now also U1.17 (PA7)
- net A8: now also U1.29 (PA8)
- net A9: now also U1.30 (PA9)
- net B0: now also U1.18 (PB0)
- net B1: now also U1.19 (PB1)
- net B10: now also U1.21 (PB10)
- net B11: now also U1.22 (PB11)
- net B12: now also U1.25 (PB12)
- net B13: now also U1.26 (PB13)
- net B14: now also U1.27 (PB14)
- net B15: now also U1.28 (PB15)
- net B2: now also U1.20 (PB2)
- net B3: now also U1.39 (PB3)
- net B4: now also U1.40 (PB4)
- net B5: now also U1.41 (PB5)
- net B6: now also U1.42 (PB6)
- net B7: now also U1.43 (PB7)
- net B8: now also U1.45 (PB8)
- net B9: now also U1.46 (PB9)
- net BOOT0: now also R1.2, U1.44 (BOOT0); no longer R1.1
- net F1: now also U1.6 (PF1)
- net GND: now also R1.1, SW2.C, U1.23 (VSS), U1.35 (VSS), U1.47 (VSS), U1.8 (VSSA), U2.1, U2.7 (GND); no longer R1.2
- net LED/DIN: now also U2.3
- net NRST: now reaches C7.1
- net NRST: now also U1.7 (NRST)
- net D+ renamed USB_D+
- net USB_D+: no longer U4.1 (I/O1)
- net D- renamed USB_D-
- net USB_D-: no longer U4.3 (I/O2)
- new net MCU_D+: U1.33 (PA12), U4.1 (I/O1)
- new net MCU_D-: U1.32 (PA11), U4.3 (I/O2)
- no-connect marks 0 -> 5
Other:
- moved on the sheet: C7, D1, D10, D100, D101, D11, D12, D13, D14, D15, D16, D17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

Commit message: :P
Connections:
- net A0: now also S34.1, S55.1, S88.1; no longer SW2.A
- net A1: now also S101.1, S33.1, S54.1, S71.1, S87.1; no longer S100.1, S31.1, S52.1, S69.1, S85.1
- net A10: now also S15.1, S2.1, S36.1, S57.1; no longer D100.1 (K), D101.1 (K), D89.1 (K), D90.1 (K), D91.1 (K), D92.1 (K), D93.1 (K), D94.1 (K), D95.1 (K), D96.1 (K), D97.1 (K), D98.1 (K), D99.1 (K)
- net A13: now also S1.1, S14.1, S35.1, S56.1, S72.1, S89.1; no longer S30.1, S51.1, S99.1
- net A14: now also D1.1 (K), D10.1 (K), D11.1 (K), D12.1 (K), D13.1 (K), D2.1 (K), D3.1 (K), D4.1 (K), D5.1 (K), D6.1 (K), D7.1 (K), D8.1 (K), D9.1 (K); no longer SW2.B
- net A3: now also S100.1, S31.1, S52.1, S69.1, S85.1; no longer S101.1, S33.1, S54.1, S71.1, S87.1
- net A4: now also S30.1, S51.1, S99.1; no longer S34.1, S55.1, S88.1
- net A5: now also S29.1, S50.1, S84.1, S98.1; no longer D1.1 (K), D10.1 (K), D11.1 (K), D12.1 (K), D13.1 (K), D2.1 (K), D3.1 (K), D4.1 (K), D5.1 (K), D6.1 (K), D7.1 (K), D8.1 (K), D9.1 (K)
- net A6: now also S28.1, S49.1, S97.1; no longer D14.1 (K), D15.1 (K), D16.1 (K), D17.1 (K), D18.1 (K), D19.1 (K), D20.1 (K), D21.1 (K), D22.1 (K), D23.1 (K), D24.1 (K), D25.1 (K), D26.1 (K), D27.1 (K), D28.1 (K), D29.1 (K), D30.1 (K), D31.1 (K), D32.1 (K), D33.1 (K), D34.1 (K)
- net A7: now also S27.1, S48.1, S68.1, S83.1, S96.1; no longer D35.1 (K), D36.1 (K), D37.1 (K), D38.1 (K), D39.1 (K), D40.1 (K), D41.1 (K), D42.1 (K), D43.1 (K), D44.1 (K), D45.1 (K), D46.1 (K), D47.1 (K), D48.1 (K), D49.1 (K), D50.1 (K), D51.1 (K), D52.1 (K), D53.1 (K), D54.1 (K), D55.1 (K)
- net A8: now also S17.1, S38.1, S4.1, S59.1, S74.1, S91.1; no longer D56.1 (K), D57.1 (K), D58.1 (K), D59.1 (K), D60.1 (K), D61.1 (K), D62.1 (K), D63.1 (K), D64.1 (K), D65.1 (K), D66.1 (K), D67.1 (K), D68.1 (K), D69.1 (K), D70.1 (K), D71.1 (K)
- net A9: now also S16.1, S3.1, S37.1, S58.1, S73.1, S90.1; no longer D72.1 (K), D73.1 (K), D74.1 (K), D75.1 (K), D76.1 (K), D77.1 (K), D78.1 (K), D79.1 (K), D80.1 (K), D81.1 (K), D82.1 (K), D83.1 (K), D84.1 (K), D85.1 (K), D86.1 (K), D87.1 (K), D88.1 (K)
- net B0: now also S13.1, S26.1, S47.1, S95.1; no longer S1.1, S14.1, S35.1, S56.1, S72.1, S89.1
- net B1: now also S12.1, S25.1, S46.1, S67.1, S82.1, S94.1; no longer S15.1, S2.1, S36.1, S57.1
- net B10: now also S10.1, S23.1, S44.1, S65.1, S80.1; no longer S11.1, S24.1, S45.1, S66.1, S81.1, S93.1
- net B11: now also S22.1, S43.1, S64.1, S79.1, S9.1; no longer S12.1, S25.1, S46.1, S67.1, S82.1, S94.1
- net B12: now also S21.1, S42.1, S63.1, S78.1, S8.1; no longer S13.1, S26.1, S47.1, S95.1
- net B13: now also S20.1, S41.1, S62.1, S7.1, S77.1, S92.1; no longer S27.1, S48.1, S68.1, S83.1, S96.1
- net B14: now also S19.1, S40.1, S6.1, S61.1, S76.1; no longer S28.1, S49.1, S97.1
- net B15: now also S18.1, S39.1, S5.1, S60.1, S75.1; no longer S29.1, S50.1, S84.1, S98.1
- net B2: now also S11.1, S24.1, S45.1, S66.1, S81.1, S93.1; no longer S16.1, S3.1, S37.1, S58.1, S73.1, S90.1
- net B3: now also SW2.A; no longer S17.1, S38.1, S4.1, S59.1, S74.1, S91.1
- net B4: now also SW2.B; no longer S18.1, S39.1, S5.1, S60.1, S75.1
- net B5: now also D100.1 (K), D101.1 (K), D89.1 (K), D90.1 (K), D91.1 (K), D92.1 (K), D93.1 (K), D94.1 (K), D95.1 (K), D96.1 (K), D97.1 (K), D98.1 (K), D99.1 (K); no longer S19.1, S40.1, S6.1, S61.1, S76.1
- net B6: now also D72.1 (K), D73.1 (K), D74.1 (K), D75.1 (K), D76.1 (K), D77.1 (K), D78.1 (K), D79.1 (K), D80.1 (K), D81.1 (K), D82.1 (K), D83.1 (K), D84.1 (K), D85.1 (K), D86.1 (K), D87.1 (K), D88.1 (K); no longer S20.1, S41.1, S62.1, S7.1, S77.1, S92.1
- net B7: now also D56.1 (K), D57.1 (K), D58.1 (K), D59.1 (K), D60.1 (K), D61.1 (K), D62.1 (K), D63.1 (K), D64.1 (K), D65.1 (K), D66.1 (K), D67.1 (K), D68.1 (K), D69.1 (K), D70.1 (K), D71.1 (K); no longer S21.1, S42.1, S63.1, S78.1, S8.1
- net B8: now also D35.1 (K), D36.1 (K), D37.1 (K), D38.1 (K), D39.1 (K), D40.1 (K), D41.1 (K), D42.1 (K), D43.1 (K), D44.1 (K), D45.1 (K), D46.1 (K), D47.1 (K), D48.1 (K), D49.1 (K), D50.1 (K), D51.1 (K), D52.1 (K), D53.1 (K), D54.1 (K), D55.1 (K); no longer S22.1, S43.1, S64.1, S79.1, S9.1
- net B9: now also D14.1 (K), D15.1 (K), D16.1 (K), D17.1 (K), D18.1 (K), D19.1 (K), D20.1 (K), D21.1 (K), D22.1 (K), D23.1 (K), D24.1 (K), D25.1 (K), D26.1 (K), D27.1 (K), D28.1 (K), D29.1 (K), D30.1 (K), D31.1 (K), D32.1 (K), D33.1 (K), D34.1 (K); no longer S10.1, S23.1, S44.1, S65.1, S80.1
